File: kicad/FancyController/PowerConnectors.kicad_sch (KiCad schematic)
At the start: 26 parts, among them J4 H-Bridge, J5 Lamp, J7 RGB, J8 Winch, J9 Motor, Q1 BC547, Q10 BUZ11, Q2 BUZ11, Q3 BC547, Q4 BUZ11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

Commit message: Changed RS232 pin mapping
Connections:
- no-connect marks 1 -> 4
Changed lines of the file:
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@@
+	)
+	(no_connect
+		(at 233.68 99.06)
+	)
+	(no_connect
+		(at 232.41 50.8)
 	)
 	(no_connect
 		(at 72.39 107.95)
 	)
+	(no_connect
+		(at 217.17 50.8)
+	)
 	(wire
