File: kicad/MainController/MainController.kicad_sch (KiCad schematic)
At the start: 21 parts, among them J1 Controller, J10 Barrel_Jack_Switch, J2 Screen, J3 JTAG, U1 ESP32-WROOM32-DevKit, U2 MAX3232, U3 L7805, U4 LTV-817, U5 LTV-817

Commit message: Fixed MainController LED power and data drivers
Parts:
- removed HS1: Heatsink_Pad, Custom_Heatsinks:Heatsink_Aavid_TO-220_H12.7mm, symbol Mechanical:Heatsink_Pad
- removed U3: L7805, Package_TO_SOT_THT:TO-220-3_Vertical, symbol Regulator_Linear:L7805
- added U7: LME78_05-1.0, Custom_Converter:Converter_DCDC_GAPTEC_LME78_05-1.0, symbol Custom_Symbols:LME78_05-1.0
- C8: value 0.1u -> 33u
Connections:
- net +12V: now also U7.1 (IN)
- net +5V: now also U7.3 (OUT)
- net GND: now also U7.2 (GND)
- no-connect marks 18 -> 17
Changed lines of the file:
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@@
 	)
 	(no_connect
-		(at 97.79 21.59)
-	)
-	(no_connect
 		(at 95.25 92.71)
 	)
@@
 	)
 	(symbol
-		(lib_id "Mechanical:Heatsink_Pad")
-		(at 97.79 19.05 0)
-		(unit 1)
-		(exclude_from_sim no)
-		(in_bom yes)
-		(on_board yes)
-		(dnp no)
-		(fields_autoplaced yes)
-		(property "Reference" "HS1"
-			(at 101.6 17.1449 0)
-			(effects
-				(font
-					(size 1.27 1.27)
-				)
-				(justify left)
-			)
-		)
-		(property "Value" "Heatsink_Pad"
-			(at 101.6 19.6849 0)
-			(effects
-				(font
-					(size 1.27 1.27)
-				)
-				(justify left)
-			)
-		)
-		(property "Footprint" "Custom_Heatsinks:Heatsink_Aavid_TO-220_H12.7mm"
-			(at 98.0948 20.32 0)
-			(effects
-				(font
-					(size 1.27 1.27)
-				)
-				(hide yes)
-			)
-		)
-		(property "Datasheet" "~"
-			(at 98.0948 20.32 0)
-			(effects
-				(font
-					(size 1.27 1.27)
-				)
-				(hide yes)
-			)
-		)
-		(property "Description" "Heatsink with electrical connection, 1 pin"
-			(at 97.79 19.05 0)
-			(effects
-				(font
-					(size 1.27 1.27)
-				)
-				(hide yes)
-			)
-		)
-		(pin "1"
-		)
-		(instances
-			(project ""
-				(path "/bf87a95b-67d4-48e1-9f7e-6bce3e771984"
-					(reference "HS1")
-					(unit 1)
-				)
-			)
-		)
-	)
-	(symbol
 		(lib_id "Device:R")
 		(at 90.17 160.02 90)
@@
 	)
 	(symbol
+		(lib_id "Custom_Symbols:LME78_05-1.0")
+		(at 97.79 33.02 0)
+		(unit 1)
+		(exclude_from_sim no)
+		(in_bom yes)
+		(on_board yes)
+		(dnp no)
+		(fields_autoplaced yes)
+		(property "Reference" "U7"
+			(at 97.79 26.67 0)
+			(effects
+				(font
+					(size 1.27 1.27)
+				)
+			)
+		)
+		(property "Value" "LME78_05-1.0"
+			(at 97.79 29.21 0)
+			(effects
+				(font
+					(size 1.27 1.27)
+				)
+			)
+		)
+		(property "Footprint" "Custom_Converter:Converter_DCDC_GAPTEC_LME78_05-1.0"
+			(at 98.425 36.83 0)
+			(effects
+				(font
+					(size 1.27 1.27)
+					(italic yes)
+				)
+				(justify left)
+				(hide yes)
+			)
+		)
+		(property "Datasheet" "https://gaptec-electronic.com/datenblaetter/LME78_1.0.pdf"
+			(at 97.79 34.29 0)
+			(effects
+				(font
+					(size 1.27 1.27)
+				)
+				(hide yes)
+			)
+		)
+		(property "Description" "Positive 1.0A 36V Linear Regulator, Fixed Output 5V, TO-220"
+			(at 97.79 33.02 0)
+			(effects
+				(font
+					(size 1.27 1.27)
+				)
+				(hide yes)
+			)
+		)
+		(pin "3"
+		)
+		(pin "1"
+		)
+		(pin "2"
+		)
+		(instances
+			(project ""
+				(path "/bf87a95b-67d4-48e1-9f7e-6bce3e771984"
+					(reference "U7")
+					(unit 1)
+				)
+			)
+		)
+	)
+	(symbol
 		(lib_id "power:+5V")
 		(at 224.79 137.16 0)
@@
 			)
 		)
-		(property "Value" "0.1u"
+		(property "Value" "33u"
 			(at 115.57 38.4809 0)
 			(effects
@@
 					(unit 1)
 				)
-			)
-		)
-	)
-	(symbol
-		(lib_id "Regulator_Linear:L7805")
-		(at 97.79 33.02 0)
-		(unit 1)
-		(exclude_from_sim no)
-		(in_bom yes)
-		(on_board yes)
-		(dnp no)
-		(fields_autoplaced yes)
-		(property "Reference" "U3"
-			(at 97.79 26.67 0)
-			(effects
-				(font
-					(size 1.27 1.27)
-				)
-			)
-		)
-		(property "Value" "L7805"
-			(at 97.79 29.21 0)
-			(effects
-				(font
-					(size 1.27 1.27)
-				)
-			)
-		)
-		(property "Footprint" "Package_TO_SOT_THT:TO-220-3_Vertical"
-			(at 98.425 36.83 0)
-			(effects
-				(font
-					(size 1.27 1.27)
-					(italic yes)
-				)
-				(justify left)
-				(hide yes)
-			)
-		)
-		(property "Datasheet" "http://www.st.com/content/ccc/resource/technical/document/datasheet/41/4f/b3/b0/12/d4/47/88/CD00000444.pdf/files/CD00000444.pdf/jcr:content/translations/en.CD00000444.pdf"
-			(at 97.79 34.29 0)
-			(effects
-				(font
-					(size 1.27 1.27)
-				)
-				(hide yes)
-			)
-		)
-		(property "Description" "Positive 1.5A 35V Linear Regulator, Fixed Output 5V, TO-220/TO-263/TO-252"
-			(at 97.79 33.02 0)
-			(effects
-				(font
-					(size 1.27 1.27)
-				)
-				(hide yes)
-			)
-		)
-		(pin "3"
-		)
-		(pin "2"
-		)
-		(pin "1"
-		)
-		(instances
-			(project "MainController"
-				(path "/bf87a95b-67d4-48e1-9f7e-6bce3e771984"
-					(reference "U3")
-					(unit 1)
-				)
